File: KiCad-Git Workshop.kicad_sch (KiCad schematic)
At the start: 1 part

Commit message: testing
Signed-off-by: blyons-dev <bthelyons@gmail.com>
Parts:
- removed R1: R, Resistor_THT:R_Axial_DIN0516_L15.5mm_D5.0mm_P20.32mm_Horizontal, symbol Device:R
Changed lines of the file:
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@@
 	(generator_version "10.0")
 	(paper "A4")
-	(symbol
-		(lib_id "Device:R")
-		(at 38.1 38.1 0)
-		(unit 1)
-		(body_style 1)
-		(exclude_from_sim no)
-		(in_bom yes)
-		(on_board yes)
-		(in_pos_files yes)
-		(dnp no)
-		(fields_autoplaced yes)
-		(property "Reference" "R1"
-			(at 40.64 36.8299 0)
-			(show_name no)
-			(do_not_autoplace no)
-			(effects
-				(font
-					(size 1.27 1.27)
-				)
-				(justify left)
-			)
-		)
-		(property "Value" "R"
-			(at 40.64 39.3699 0)
-			(show_name no)
-			(do_not_autoplace no)
-			(effects
-				(font
-					(size 1.27 1.27)
-				)
-				(justify left)
-			)
-		)
-		(property "Footprint" "Resistor_THT:R_Axial_DIN0516_L15.5mm_D5.0mm_P20.32mm_Horizontal"
-			(at 36.322 38.1 90)
-			(hide yes)
-			(show_name no)
-			(do_not_autoplace no)
-			(effects
-				(font
-					(size 1.27 1.27)
-				)
-			)
-		)
-		(property "Datasheet" ""
-			(at 38.1 38.1 0)
-			(hide yes)
-			(show_name no)
-			(do_not_autoplace no)
-			(effects
-				(font
-					(size 1.27 1.27)
-				)
-			)
-		)
-		(property "Description" "Resistor"
-			(at 38.1 38.1 0)
-			(hide yes)
-			(show_name no)
-			(do_not_autoplace no)
-			(effects
-				(font
-					(size 1.27 1.27)
-				)
-			)
-		)
-		(pin "1"
-		)
-		(pin "2"
-		)
-		(instances
-			(project "KiCad-Git Workshop"
-				(path "/2560e339-23aa-4fe7-8757-a9286f7a6852"
-					(reference "R1")
-					(unit 1)
-				)
-			)
-		)
-	)
 	(sheet_instances
 		(path "/"

Commit message: Signed-off-by: blyons-dev <bthelyons@gmail.com>
Other:
- note added: "Congratulations! You have successfully pulled the KiCad files from the GitHub repository! Yippee! The next step is to make a change to the schematic and/or the layout and push the changes to a new branch of the repository. Step-by-Step Instructions: 1. Change the schematic/layout 2. Go into the layout editor (The Git plugin interface can only be accessed through the layout editor for reasons) 3. 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"
Changed lines of the file:
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@@
 	(generator_version "10.0")
 	(paper "A4")
+	(text "Congratulations!\nYou have successfully pulled the KiCad files from the GitHub repository! Yippee!\nThe next step is to make a change to the schematic and/or the layout and push the changes to a new branch of the repository.\n\nStep-by-Step Instructions:\n1. Change the schematic/layout\n2. Go into the layout editor (The Git plugin interface can only be accessed through the layout editor for reasons)\n3. Launch the Git plugin interface\n4. Create a new branch and name it first_initial-last_name\n5. Make sure all of your changes are unstaged by clicking Rescan\n6. Click Stage Changed to prepare your changes for a Commit\n7. Write in the Commit Message what you changed\n8. Click Sign-Off for formalities\n9. Click Commit\n10. Click Push to push the changes to the branch you just created"
+		(exclude_from_sim no)
+		(at 127 63.754 0)
+		(effects
+			(font
+				(size 1.27 1.27)
+			)
+		)
+	)
 	(sheet_instances
 		(path "/"

Commit message: Prepared Initial Instructions for Workshop
Signed-off-by: blyons-dev <bthelyons@gmail.com>
Other:
- note added: "Congratulations! You have successfully pulled the KiCad files from the GitHub repository! Yippee! The next step is to make a change to the schematic and/or the layout and push the changes to a new branch of the repository. Step-by-Step Instructions: 1. Change the schematic/layout and save the file after changing it 2. Go into the layout editor (The Git plugin interface can only be accessed throug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"
- note removed: "Congratulations! You have successfully pulled the KiCad files from the GitHub repository! Yippee! The next step is to make a change to the schematic and/or the layout and push the changes to a new branch of the repository. Step-by-Step Instructions: 1. Change the schematic/layout 2. Go into the layout editor (The Git plugin interface can only be accessed through the layout editor for reasons) 3. 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"
Changed lines of the file:
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@@
 	(generator_version "10.0")
 	(paper "A4")
-	(text "Congratulations!\nYou have successfully pulled the KiCad files from the GitHub repository! Yippee!\nThe next step is to make a change to the schematic and/or the layout and push the changes to a new branch of the repository.\n\nStep-by-Step Instructions:\n1. Change the schematic/layout\n2. Go into the layout editor (The Git plugin interface can only be accessed through the layout editor for reasons)\n3. Launch the Git plugin interface\n4. Create a new branch and name it first_initial-last_name\n5. Make sure all of your changes are unstaged by clicking Rescan\n6. Click Stage Changed to prepare your changes for a Commit\n7. Write in the Commit Message what you changed\n8. Click Sign-Off for formalities\n9. Click Commit\n10. Click Push to push the changes to the branch you just created"
+	(text "Congratulations!\nYou have successfully pulled the KiCad files from the GitHub repository! Yippee!\nThe next step is to make a change to the schematic and/or the layout and push the changes to a new branch of the repository.\n\nStep-by-Step Instructions:\n1. Change the schematic/layout and save the file after changing it\n2. Go into the layout editor (The Git plugin interface can only be accessed through the layout editor for reasons)\n3. Launch the Git plugin interface\n4. Create a new branch and name it first_initial-last_name\n5. Make sure all of your changes are unstaged by clicking Rescan\n6. Click Stage Changed to prepare your changes for a Commit\n7. Write in the Commit Message what you changed\n8. Click Sign-Off for formalities\n9. Click Commit\n10. Click Push to push the changes to the branch you just created\n\nThis is the project workflow of using Git with KiCad!\nAll that is left to do is to go back into GitHub and create a Pull Request if you are done making changes on your branch and it is ready to be merged with the main"
 		(exclude_from_sim no)
-		(at 127 63.754 0)
+		(at 148.844 95.758 0)
 		(effects
 			(font
-				(size 1.27 1.27)
+				(size 1.905 1.905)
 			)
 		)

Commit message: Included step in instruction to identify oneself
Signed-off-by: blyons-dev <bthelyons@gmail.com>
Other:
- note added: "2Congratulations! You have successfully pulled the KiCad files from the GitHub repository! Yippee! The next step is to make a change to the schematic and/or the layout and push the changes to a new branch of the repository. Step-by-Step Instructions: 1. Change the schematic/layout and save the file after changing it 2. Go into the layout editor (The Git plugin interface can only be accessed throu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"
- note removed: "Congratulations! You have successfully pulled the KiCad files from the GitHub repository! Yippee! The next step is to make a change to the schematic and/or the layout and push the changes to a new branch of the repository. Step-by-Step Instructions: 1. Change the schematic/layout and save the file after changing it 2. Go into the layout editor (The Git plugin interface can only be accessed throug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"
Changed lines of the file:
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@@
 	(generator_version "10.0")
 	(paper "A4")
-	(text "Congratulations!\nYou have successfully pulled the KiCad files from the GitHub repository! Yippee!\nThe next step is to make a change to the schematic and/or the layout and push the changes to a new branch of the repository.\n\nStep-by-Step Instructions:\n1. Change the schematic/layout and save the file after changing it\n2. Go into the layout editor (The Git plugin interface can only be accessed through the layout editor for reasons)\n3. Launch the Git plugin interface\n4. Create a new branch and name it first_initial-last_name\n5. Make sure all of your changes are unstaged by clicking Rescan\n6. Click Stage Changed to prepare your changes for a Commit\n7. Write in the Commit Message what you changed\n8. Click Sign-Off for formalities\n9. Click Commit\n10. Click Push to push the changes to the branch you just created\n\nThis is the project workflow of using Git with KiCad!\nAll that is left to do is to go back into GitHub and create a Pull Request if you are done making changes on your branch and it is ready to be merged with the main"
+	(text "2Congratulations!\nYou have successfully pulled the KiCad files from the GitHub repository! Yippee!\nThe next step is to make a change to the schematic and/or the layout and push the changes to a new branch of the repository.\n\nStep-by-Step Instructions:\n1. Change the schematic/layout and save the file after changing it\n2. Go into the layout editor (The Git plugin interface can only be accessed through the layout editor for reasons)\n3. Launch the Git plugin interface\n4. Set your User Name and Email under Edit->Options so that the plugin knows who you are and will let you commit\n5. Create a new branch and name it first_initial-last_name\n6. Make sure all of your changes are unstaged by clicking Rescan\n7. Click Stage Changed to prepare your changes for a Commit\n8. Write in the Commit Message what you changed\n9. Click Sign-Off for formalities\n10. Click Commit\n11. Click Push to push the changes to the branch you just created\n\nThis is the project workflow of using Git with KiCad!\nAll that is left to do is to go back into GitHub and create a Pull Request if you are done making changes on your branch and it is ready to be merged with the main"
 		(exclude_from_sim no)
 		(at 148.844 95.758 0)

Commit message: Removed a 2
fixed the message
Other:
- note added: "Congratulations! You have successfully pulled the KiCad files from the GitHub repository! Yippee! The next step is to make a change to the schematic and/or the layout and push the changes to a new branch of the repository. Step-by-Step Instructions: 1. Change the schematic/layout and save the file after changing it 2. Go into the layout editor (The Git plugin interface can only be accessed throug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"
- note removed: "2Congratulations! You have successfully pulled the KiCad files from the GitHub repository! Yippee! The next step is to make a change to the schematic and/or the layout and push the changes to a new branch of the repository. Step-by-Step Instructions: 1. Change the schematic/layout and save the file after changing it 2. Go into the layout editor (The Git plugin interface can only be accessed throu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"
Changed lines of the file:
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@@
 	(generator_version "10.0")
 	(paper "A4")
-	(text "2Congratulations!\nYou have successfully pulled the KiCad files from the GitHub repository! Yippee!\nThe next step is to make a change to the schematic and/or the layout and push the changes to a new branch of the repository.\n\nStep-by-Step Instructions:\n1. Change the schematic/layout and save the file after changing it\n2. Go into the layout editor (The Git plugin interface can only be accessed through the layout editor for reasons)\n3. Launch the Git plugin interface\n4. Set your User Name and Email under Edit->Options so that the plugin knows who you are and will let you commit\n5. Create a new branch and name it first_initial-last_name\n6. Make sure all of your changes are unstaged by clicking Rescan\n7. Click Stage Changed to prepare your changes for a Commit\n8. Write in the Commit Message what you changed\n9. Click Sign-Off for formalities\n10. Click Commit\n11. Click Push to push the changes to the branch you just created\n\nThis is the project workflow of using Git with KiCad!\nAll that is left to do is to go back into GitHub and create a Pull Request if you are done making changes on your branch and it is ready to be merged with the main"
+	(text "Congratulations!\nYou have successfully pulled the KiCad files from the GitHub repository! Yippee!\nThe next step is to make a change to the schematic and/or the layout and push the changes to a new branch of the repository.\n\nStep-by-Step Instructions:\n1. Change the schematic/layout and save the file after changing it\n2. Go into the layout editor (The Git plugin interface can only be accessed through the layout editor for reasons)\n3. Launch the Git plugin interface\n4. Set your User Name and Email under Edit->Options so that the plugin knows who you are and will let you commit\n5. Create a new branch and name it first_initial-last_name\n6. Make sure all of your changes are unstaged by clicking Rescan\n7. Click Stage Changed to prepare your changes for a Commit\n8. Write in the Commit Message what you changed\n9. Click Sign-Off for formalities\n10. Click Commit\n11. Click Push to push the changes to the branch you just created\n\nThis is the project workflow of using Git with KiCad!\nAll that is left to do is to go back into GitHub and create a Pull Request if you are done making changes on your branch and it is ready to be merged with the main"
 		(exclude_from_sim no)
 		(at 148.844 95.758 0)
